Commit message: v2

File: uthai_description/urdf/uthai.urdf.xacro (robot description, xacro)
@@ -3,4 +3,5 @@
     xmlns:xacro="http://www.ros.org/wiki/xacro">
     <xacro:property name="pi" value="3.141592654"/>
+    <xacro:property name="fixed_body" value="False"/>
     <!-- Import xacro file -->
     <xacro:include filename="$(find uthai_description)/urdf/materials.xacro" />
@@ -12,10 +13,12 @@
     <xacro:include filename="$(find uthai_description)/urdf/uthai.gazebo.xacro" />
     <!-- Used for fixing robot -->
-    <!--<link name="world"></link>
-    <joint name="world_fixed" type="fixed">
-        <origin xyz="0 0 0.764" rpy="0 0 0"/>
-        <parent link="world"/>
-        <child link="base_link"/>
-    </joint> -->
+    <xacro:if value="${fixed_body == True}">
+        <link name="world"></link>
+        <joint name="world_fixed" type="fixed">
+            <origin xyz="0 0 0." rpy="0 0 0"/>
+            <parent link="world"/>
+            <child link="base_link"/>
+        </joint>
+    </xacro:if>
     <link name="base_link"></link>
     <joint name="base_fixed" type="fixed">

File: uthai_description/urdf/uthai.urdf_exercise.xacro (robot description, xacro)
@@ -3,4 +3,7 @@
     xmlns:xacro="http://www.ros.org/wiki/xacro">
     <xacro:property name="pi" value="3.141592654"/>
+    <!-- exercise:  -->
+    <xacro:property name="fixed_body" value="True"/>
+    <!-- end exercise:  -->
     <!-- Import xacro file -->
     <xacro:include filename="$(find uthai_description)/urdf/materials.xacro" />
@@ -12,10 +15,12 @@
     <xacro:include filename="$(find uthai_description)/urdf/uthai.gazebo.xacro" />
     <!-- Used for fixing robot -->
-    <!--<link name="world"></link>
-    <joint name="world_fixed" type="fixed">
-        <origin xyz="0 0 0.764" rpy="0 0 0"/>
-        <parent link="world"/>
-        <child link="base_link"/>
-    </joint> -->
+    <xacro:if value="${fixed_body == True}">
+        <link name="world"></link>
+        <joint name="world_fixed" type="fixed">
+            <origin xyz="0 0 0." rpy="0 0 0"/>
+            <parent link="world"/>
+            <child link="base_link"/>
+        </joint>
+    </xacro:if>
     <link name="base_link"></link>
     <joint name="base_fixed" type="fixed">
@@ -44,5 +49,5 @@
     <link name="imu_link"></link>
     <!-- leg link -->
-    <xacro:uthai_right_leg parent="base_footprint" dxl_effort="10000" dxl_speed="3"/>
-    <xacro:uthai_left_leg parent="base_footprint" dxl_effort="10000" dxl_speed="3"/>
+    <xacro:uthai_right_leg parent="base_footprint" dxl_effort="1000" dxl_speed="3"/>
+    <xacro:uthai_left_leg parent="base_footprint" dxl_effort="1000" dxl_speed="3"/>
 </robot>
